File: marimba.sch (KiCad schematic (older format))
At the start: 53 parts, among them J1 CONN_02X16, U1 LM324, U2 LM324, U3 LM324, U4 LM324

Commit message: demux + µc
Parts:
- added U5: HCF4067B, symbol HCF4067B
- added U6: ATMEGA328P-MMH, MLF/QFN28, symbol ATMEGA328P-MMH
Connections:
- net labels added: +5V
- net labels removed: +9V
- wire segments 221 -> 261
Other:
- note added: "DEMUX"
- note added: "INPUT"
- note added: "PREAMPS"

Commit message: midi output && xtal
Parts:
- added C1, C2: 18p, symbol CP1_Small
- added C3: 100n, symbol CP1_Small
- added J2: DIN_5, symbol DIN_5
- added R33: 220, symbol R
- added Y1: 8M, symbol Crystal_Small
Connections:
- wire segments 261 -> 283
