File: electric/marimba.sch (KiCad schematic (older format))
At the start: 61 parts, among them J1 CONN_02X16, J2 DIN_5, U1 LM324, U2 LM324, U3 LM324, U4 LM324, U5 HCF4067B, U6 ATMEGA328P-MMH, Y1 8M

Commit message: missing resistor values && power supply
Parts:
- added C4: 10u, symbol CP
- added C5, C6: 100n, symbol C
- added D1: 1N4001, symbol D
- added J3: BARREL_JACK, symbol BARREL_JACK
- added U7: 7805, symbol 7805
- R21, R22, R23, R24, R25, R26, R27, R28, R29, R30, R31, R32, R5, R6, R7, R8: value R -> 1M
Connections:
- wire segments 283 -> 297
Other:
- note added: "MIDI OUT"
- note added: "POWER SUPPLY"
- moved on the sheet: J1, R10, R11, R12, R13, R14, R15, R16, R17, R18, R19, R20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
